File: elec/layout/default/rp2040-custom.kicad_pcb (KiCad board)
At the start: 2 copper layers, 225.7 x 100.8 mm, 0 parts

Commit message: Currently broken, but pushing for review
Parts:
- added C1: Multilayer Ceramic Capacitors MLCC - SMD/SMT 20pF 50V 0402 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, lib:C0402, F.Cu at (126.0, 87.4)
- added C10: Multilayer Ceramic Capacitors MLCC - SMD/SMT 100nF 10V 0402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, lib:C0402, F.Cu at (126.3, 101.5)
- added C11: Multilayer Ceramic Capacitors MLCC - SMD/SMT 100nF 10V 0402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, lib:C0402, F.Cu at (126.3, 100.2)
- added C12: Multilayer Ceramic Capacitors MLCC - SMD/SMT 1uF 6.3V 0402 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, lib:C0402, F.Cu at (126.3, 98.9)
- added C13: Multilayer Ceramic Capacitors MLCC - SMD/SMT 1uF 6.3V 0402 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, lib:C0402, F.Cu at (143.6, 86.6)
- added C14: Multilayer Ceramic Capacitors MLCC - SMD/SMT 1uF 6.3V 0402 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, lib:C0402, F.Cu at (123.3, 94.7)
- added C2: Multilayer Ceramic Capacitors MLCC - SMD/SMT 20pF 50V 0402 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, lib:C0402, F.Cu at (123.3, 85.0)
- added C3: Multilayer Ceramic Capacitors MLCC - SMD/SMT 100nF 10V 0402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, lib:C0402, F.Cu at (130.9, 94.7)
- added C4: Multilayer Ceramic Capacitors MLCC - SMD/SMT 100nF 10V 0402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, lib:C0402, F.Cu at (129.7, 94.7)
- added C5: Multilayer Ceramic Capacitors MLCC - SMD/SMT 100nF 10V 0402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, lib:C0402, F.Cu at (128.4, 94.7)
- added C6: Multilayer Ceramic Capacitors MLCC - SMD/SMT 100nF 10V 0402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, lib:C0402, F.Cu at (127.1, 94.7)
- added C7: Multilayer Ceramic Capacitors MLCC - SMD/SMT 100nF 10V 0402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, lib:C0402, F.Cu at (125.9, 94.7)
- added C8: Multilayer Ceramic Capacitors MLCC - SMD/SMT 1uF 6.3V 0402 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, lib:C0402, F.Cu at (124.6, 94.7)
- added C9: Multilayer Ceramic Capacitors MLCC - SMD/SMT 100nF 10V 0402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, lib:C0402, F.Cu at (126.3, 102.7)
- added R1: Chip Resistor - Surface Mount 1KOhms ±5% 1/16W 0402 RoHS, lib:R0402, F.Cu at (121.9, 94.7)
- added R2: Chip Resistor - Surface Mount 27KOhms ±5% 1/16W 0402 RoHS, lib:R0402, F.Cu at (140.6, 93.0)
- added R3: Chip Resistor - Surface Mount 27KOhms ±5% 1/16W 0402 RoHS, lib:R0402, F.Cu at (141.9, 93.0)
- added R4: Chip Resistor - Surface Mount 10KOhms ±5% 1/16W 0402 RoHS, lib:R0402, F.Cu at (139.3, 93.0)
- added R5: Chip Resistor - Surface Mount 10KOhms ±5% 1/16W 0402 RoHS, lib:R0402, F.Cu at (137.9, 93.0)
- added R6: Chip Resistor - Surface Mount 18KOhms ±5% 1/16W 0402 RoHS, lib:R0402, F.Cu at (136.5, 93.0)
- added R7: Chip Resistor - Surface Mount 10KOhms ±5% 1/16W 0402 RoHS, lib:R0402, F.Cu at (135.1, 93.0)
- added R8: Chip Resistor - Surface Mount 4.7KOhms ±5% 1/16W 0402 RoHS, lib:R0402, F.Cu at (143.6, 88.0)
- added R9: Chip Resistor - Surface Mount 4.7KOhms ±5% 1/16W 0402 RoHS, lib:R0402, F.Cu at (143.6, 89.4)
- added U1: , lib:LQFN-56_L7.0-W7.0-P0.4-EP, F.Cu at (132.3, 100.6)
- added U2: , lib:OSC-SMD_4P-L3.2-W2.5-BL, F.Cu at (123.3, 88.0)
- added U3: , lib:SOIC-8_L5.3-W5.3-P1.27-LS8.0-BL, F.Cu at (142.6, 100.5)
- added U4: , lib:SOT-23-5_L3.0-W1.7-P0.95-LS2.8-BL, F.Cu at (140.2, 88.0)
- added U5: , lib:USB-C-SMD_KH-TYPE-C-16P, F.Cu at (132.6, 87.9)
Routing:
- net vcc-4: track 0.00 -> 21.8 mm
- net cs: track 0.00 -> 17.9 mm
- net io1: track 0.00 -> 16.1 mm
- net CC1: track 0.00 -> 14.9 mm
- net vcc: track 0.00 -> 13.8 mm
- net io2: track 0.00 -> 11.3 mm
- net vcc-3: track 0.00 -> 10.0 mm
- net xout: track 0.00 -> 9.59 mm
- net gnd: track 0.00 -> 8.24 mm
- net vcc-1: track 0.00 -> 5.97 mm
- net io3: track 0.00 -> 3.64 mm
- net io0: track 0.00 -> 3.44 mm
- net sck: track 0.00 -> 3.28 mm
- net vcc-2: track 0.00 -> 2.31 mm
- net gnd-4: track 0.00 -> 1.91 mm
- added copper zone on B.Cu, net gnd
Other:
- board size 225.7 x 100.8 mm -> 40 x 40 mm
